Commit message: add class at ball localization node and modified urdf

File: fibot_description/urdf/fibot_robot_demo_joint_test.urdf (robot description, URDF)
Before this commit: robot rehri, 8 links, 7 joints
Links:
- link caster: geometry collision sphere radius=0.075; visual sphere radius=0.075
Joints:
- joint base_joint: origin xyz=0 0 0.135 rpy=0 0 0 -> xyz=0 0 0.15 rpy=0 0 0
- joint caster_joint: origin xyz=0.3 0.0 -0.07 rpy=0.0 0.0 0.0 -> xyz=0.3 0.0 -0.075 rpy=0.0 0.0 0.0

Commit message: update ball detection node and urdf

File: fibot_description/urdf/fibot_robot_demo_joint_test.urdf (robot description, URDF)
Before this commit: robot rehri, 8 links, 7 joints
Links:
- added link camera_link_fixed, mass 0.1; collision box size=0.1 0.1 0.05; visual box size=0.1 0.1 0.05
Joints:
- added joint camera_joint_fixed: type fixed, parent yaw_camera, child camera_link_fixed, origin xyz=0.0 0.0 0.0 rpy=0 0.0 0, axis 0.0 1.0 0.0, limit lower=-1.57 upper=1.57 effort=100.0 velocity=0.5
- joint camera_joint: origin xyz=0.0 0 0.0 rpy=3.14 2.61799 3.14 -> xyz=0.0 0.0 0.0 rpy=0.0 0.0 0.0; parent yaw_camera -> camera_link_fixed
- joint caster_joint: origin xyz=0.3 0.0 -0.075 rpy=0.0 0.0 0.0 -> xyz=0.3 0.0 -0.0750 rpy=0.0 0.0 0.0
- joint yaw_camera_joint: origin xyz=0.35 0 0.5 rpy=0.0 0.0 0.0 -> xyz=0.35 0.0 0.50 rpy=0.0 0.0 0.0

Commit message: add traj node and add code for vary angle

File: fibot_description/urdf/fibot_robot_demo_joint_test.urdf (robot description, URDF)
Before this commit: robot rehri, 9 links, 8 joints
Links:
- link camera: geometry visual box size=0.1 0.1 0.05
- link camera_link_fixed: geometry visual box size=0.1 0.1 0.05
- link yaw_camera: geometry visual box size=0.1 0.1 0.05
Joints:
- joint camera_joint: origin xyz=0.0 0.0 0.0 rpy=0.0 0.0 0.0 -> xyz=0.0 0.0 0.13 rpy=0.0 0.0 0.0

Commit message: IPM from tf2

File: fibot_description/urdf/fibot_robot_demo_joint_test.urdf (robot description, URDF)
Before this commit: robot rehri, 9 links, 8 joints
Links:
- link base: mass 1 -> 5
- link camera: mass 0.1 -> 1.0; geometry collision box size=0.1 0.1 0.05; visual box size=0.1 0.1 0.05
- link camera_link_fixed: mass 0.1 -> 1.0
- link yaw_camera: mass 0.1 -> 1.0
Joints:
- joint camera_joint: limit lower=-1.57 upper=1.57 effort=100.0 velocity=0.5 -> lower=-1.57 upper=1.57 effort=10000.0 velocity=0.1
- joint camera_joint_fixed: limit lower=-1.57 upper=1.57 effort=100.0 velocity=0.5 -> lower=-3.14 upper=3.14 effort=100000.0 velocity=0.5
- joint yaw_camera_joint: limit lower=-3.14 upper=3.14 effort=100.0 velocity=0.5 -> lower=-3.14 upper=3.14 effort=10000.0 velocity=0.5
