Commit message: Update fibot_xacro.urdf.xacro
add macro

File: fibot_description/urdf/fibot_xacro.urdf.xacro (robot description, xacro)
@@ -59,77 +59,52 @@
     <xacro:base_inertial mass="0.291"/>
   </link>
-  <link name="right_hip_link">
-    <visual>
-      <origin xyz="0 0 0"/>
-      <!-- <origin xyz="0.0305 0  ${-(base_height+right_hip_height)/2}"/> -->
-      <geometry>
-        <box size="${right_hip_width} ${right_hip_length} ${right_hip_height}"/>
-      </geometry>
-      <material name="black"/>
-    </visual>
-    <collision>
-      <origin xyz="0 0 0"/>
-      <!-- <origin xyz="0.0305 0  ${-(base_height+right_hip_height)/2}"/> -->
-      <geometry>
-        <box size="${right_hip_width} ${right_hip_length} ${right_hip_height}"/>
-      </geometry>
-    </collision>
-  </link>
-  <joint name="base_link_to_rigth_hip_link" type="continuous">
-    <parent link="base_link"/>
-    <child link="right_hip_link"/>
-    <!-- <origin xyz="0 0.0305 ${base_height/2}"/> -->
-    <origin xyz="0.0305 0 ${-(base_height+right_hip_height)/2}"/>
-  </joint>
-  <link name="right_bum_link">
-    <visual>
-      <origin xyz="0 -0.0221 0"/>
-      <geometry>
-        <box size="${right_bum_width} ${right_bum_length} ${right_bum_height}"/>
-      </geometry>
-      <material name="black"/>
-    </visual>
-    <collision>
-      <geometry>
-        <box size="${right_bum_width} ${right_bum_length} ${right_bum_height}"/>
-      </geometry>
-    </collision>
-  </link>
-  <joint name="right_hip_to_right_bum" type="fixed">
-    <parent link="right_hip_link"/>
-    <child link="right_bum_link"/>
-    <origin xyz="0 0 ${-right_bum_height/2}"/>
-  </joint>
-  <!-- <link name="right_foot">
-    <visual>
-      <origin xyz="0 0.5 ${foot_height/2}" />
-      <geometry>
-        <box size="${foot_width} ${foot_length} ${foot_height}"/>
-      </geometry>
-      <material name="black"/>
-    </visual>
-  </link>
-  <link name="upper_right_foot">
-    <visual>
-      <origin xyz="0 0 ${foot_height/2}" />
-      <geometry>
-        <box size="${upper_foot_width} ${upper_foot_length} ${upper_foot_height}"/>
-      </geometry>
-      <material name="blue"/>
-    </visual>
-  </link>
-  <joint name="right_foot_to_upper_right_foot" type="fixed">
-    <parent link="upper_right_foot"/>
-    <child link="right_foot"/>
-    <origin xyz="0 0 ${foot_height/2}"/>
-  </joint>
-  <link name="left_foot">
-    <visual>
-      <origin xyz="0 -0.5 ${foot_height/2}"/>
-      <geometry>
-        <box size="${foot_width} ${foot_length} ${foot_height}"/>
-      </geometry>
-      <material name="black"/>
-    </visual>
-  </link> -->
+  <!-- ############################################################## macro robot hip ####################################################-->
+  <xacro:macro name="hip" params='prefix reflect'>
+    <link name="${prefix}_hip_link">
+      <visual>
+        <origin xyz="0 0 0"/>
+        <geometry>
+          <box size="${right_hip_width} ${right_hip_length} ${right_hip_height}"/>
+        </geometry>
+        <material name="black"/>
+      </visual>
+      <collision>
+        <origin xyz="0 0 0"/>
+        <geometry>
+          <box size="${right_hip_width} ${right_hip_length} ${right_hip_height}"/>
+        </geometry>
+      </collision>
+    </link>
+    <joint name="base_link_to_${prefix}_hip_link" type="continuous">
+      <parent link="base_link"/>
+      <child link="${prefix}_hip_link"/>
+      <origin xyz="${0.0305*reflect} 0 ${-(base_height+right_hip_height)/2}"/>
+    </joint>
+  </xacro:macro>
+  <xacro:hip prefix="right" reflect="1"/>
+  <xacro:hip prefix="left" reflect="-1"/>
+  <!-- ############################################################## macro robot hip ####################################################-->
+  <xacro:macro name="bum" params="prefix">
+    <link name="${prefix}_bum_link">
+      <visual>
+        <origin xyz="0 -0.0221 0"/>
+        <geometry>
+          <box size="${right_bum_width} ${right_bum_length} ${right_bum_height}"/>
+        </geometry>
+        <material name="black"/>
+      </visual>
+      <collision>
+        <geometry>
+          <box size="${right_bum_width} ${right_bum_length} ${right_bum_height}"/>
+        </geometry>
+      </collision>
+    </link>
+    <joint name="${prefix}_hip_to_${prefix}_bum" type="fixed">
+      <parent link="${prefix}_hip_link"/>
+      <child link="${prefix}_bum_link"/>
+      <origin xyz="0 0 ${-right_bum_height/2}"/>
+    </joint>
+  </xacro:macro>
+  <xacro:bum prefix="right"/>
+  <xacro:bum prefix="left"/>
 </robot>

Commit message: Update fibot_xacro.urdf.xacro
add lower leg

File: fibot_description/urdf/fibot_xacro.urdf.xacro (robot description, xacro)
@@ -1,10 +1,5 @@
 <?xml version="1.0"?>
 <robot name="macroed" xmlns:xacro="http://ros.org/wiki/xacro">
-  <!-- <xacro:property name="leglen" value="0.6" />
-  <xacro:property name="polelen" value="0.2" />
-  <xacro:property name="bodylen" value="0.6" />
-  <xacro:property name="baselen" value="0.4" />
-  <xacro:property name="wheeldiam" value="0.07" />
-  <xacro:property name="pi" value="3.1415" /> -->
+ <!-- Unit in this file is determine in meter and kilogram -->
 <!-- ###########################################################set up property #################################################################-->
   <xacro:property name="base_width" value="0.156" />
@@ -24,4 +19,13 @@
   <xacro:property name="right_bum_length" value="0.0922"/>
   <xacro:property name="right_bum_height" value="0.06"/>
+  <xacro:property name="upper_leg_width" value="0.054"/>
+  <xacro:property name="upper_leg_length" value="0.03"/>
+  <xacro:property name="upper_leg_height" value="0.1553"/>
+  <xacro:property name="lower_leg_width" value="0.054"/>
+  <xacro:property name="lower_leg_length" value="0.03"/>
+  <xacro:property name="lower_leg_height" value="0.16039"/>
+  <xacro:property name="ankel_width" value="0.048"/>
+  <xacro:property name="ankel_length" value="0.0922"/>
+  <xacro:property name="ankel_height" value="0.06"/>
   <xacro:property name="pi" value="3.1415"/>
 <!-- ###########################################################set up property #################################################################-->
@@ -35,4 +39,16 @@
   <material name="white">
     <color rgba="1 1 1 1"/>
+  </material>
+  <material name="red">
+  <color rgba="1 0 0 1"/>
+  </material>
+  <material name="yellow">
+  <color rgba="1 1 0 1"/>
+  </material>
+  <material name="turqouise">
+  <color rgba="0 1 1 1"/>
+  </material>
+  <material name="violet">
+  <color rgba="1 0 1 1"/>
   </material>
 <!-- ###########################################################set up material #################################################################-->
@@ -43,7 +59,8 @@
     </inertial>
   </xacro:macro>
+<!-- add foot_print -->
+<!-- add foot_print -->
   <link name="base_link">
     <visual>
-      <!-- <origin xyz="0 0 ${base_height_pos}"/> -->
       <geometry>
         <box size="${base_width} ${base_length} ${base_height}"/>
@@ -52,5 +69,4 @@
     </visual>
     <collision>
-      <!-- <origin xyz="0 0 ${base_height_pos}"/> -->
       <geometry>
         <box size="${base_width} ${base_length} ${base_height}"/>
@@ -59,5 +75,5 @@
     <xacro:base_inertial mass="0.291"/>
   </link>
-  <!-- ############################################################## macro robot hip ####################################################-->
+  <!-- ############################################################## macro robot's hip ####################################################-->
   <xacro:macro name="hip" params='prefix reflect'>
     <link name="${prefix}_hip_link">
@@ -84,6 +100,6 @@
   <xacro:hip prefix="right" reflect="1"/>
   <xacro:hip prefix="left" reflect="-1"/>
-  <!-- ############################################################## macro robot hip ####################################################-->
-  <xacro:macro name="bum" params="prefix">
+  <!-- ############################################################## macro robot's bum ####################################################-->
+  <xacro:macro name="bum" params="prefix ">
     <link name="${prefix}_bum_link">
       <visual>
@@ -105,6 +121,81 @@
       <origin xyz="0 0 ${-right_bum_height/2}"/>
     </joint>
+      <!-- origin may been wong because 'z' may be not bum height divine by 2, it might increse in 'z' axis -->
   </xacro:macro>
   <xacro:bum prefix="right"/>
   <xacro:bum prefix="left"/>
+  <!--########################################################## macro robot's upper leg #######################################################-->
+  <xacro:macro name="upper_leg" params="prefix">
+    <link name="${prefix}_upper_leg_link">
+      <visual>
+        <origin xyz="0 0 ${-upper_leg_height/2}"/>
+        <geometry>
+          <box size="${upper_leg_width} ${upper_leg_length} ${upper_leg_height}"/>
+        </geometry>
+        <material name="red"/>
+      </visual>
+      <collision>
+        <geometry>
+          <box size="${upper_leg_width} ${upper_leg_length} ${upper_leg_height}"/>
+        </geometry>
+      </collision>
+    </link>
+    <joint name="${prefix}_bum_to_${prefix}_upper_leg" type="fixed">
+      <parent link="${prefix}_bum_link"/>
+      <child link="${prefix}_upper_leg_link"/>
+      <origin xyz="0 0 0"/>
+      <!-- origin must be the same with bum joint -->
+    </joint>
+  </xacro:macro>
+  <xacro:upper_leg prefix="right"/>
+  <xacro:upper_leg prefix="left"/>
+  <!--########################################################## macro robot's lower leg #######################################################-->
+  <xacro:macro name="lower_leg" params="prefix">
+    <link name="${prefix}_lower_leg_link">
+      <visual>
+        <origin xyz="0 0 ${-lower_leg_height/2}"/>
+        <geometry>
+          <box size="${lower_leg_width} ${lower_leg_length} ${lower_leg_height}"/>
+        </geometry>
+        <material name="yellow"/>
+      </visual>
+      <collision>
+        <geometry>
+          <box size="${lower_leg_width} ${lower_leg_length} ${lower_leg_height}"/>
+        </geometry>
+      </collision>
+    </link>
+  <joint name="${prefix}_upper_leg_to_${prefix}_lower_leg" type="fixed">
+    <parent link="${prefix}_upper_leg_link"/>
+    <child link="${prefix}_lower_leg_link"/>
+    <origin xyz="0 0 ${-upper_leg_height}"/>
+  </joint>
+  </xacro:macro>
+  <xacro:lower_leg prefix="right"/>
+  <xacro:lower_leg prefix="left"/>
+  <!--########################################################## macro robot's ankel #######################################################-->
+  <xacro:macro name="ankel" params="prefix">
+    <link name="${prefix}_ankel_link">
+      <visual>
+        <origin xyz="0 -0.0221 0"/>
+        <geometry>
+          <box size="${ankel_width} ${ankel_length} ${ankel_height}"/>
+        </geometry>
+        <material name="turqouise"/>
+      </visual>
+      <collision>
+        <geometry>
+          <box size="${ankel_width} ${ankel_length} ${ankel_height}"/>
+        </geometry>
+      </collision>
+    </link>
+    <joint name="${prefix}_lower_leg_to_${prefix}_ankel" type="fixed">
+      <parent link="${prefix}_lower_leg_link"/>
+      <child link="${prefix}_ankel_link"/>
+      <origin xyz="0 0 ${-lower_leg_height}"/>
+    </joint>
+  </xacro:macro>
+  <xacro:ankel prefix="right"/>
+  <xacro:ankel prefix="left"/>
 </robot>
+  <!--########################################################## macro robot's upper foot #######################################################-->

Commit message: Update fibot_xacro.urdf.xacro
add ankel

File: fibot_description/urdf/fibot_xacro.urdf.xacro (robot description, xacro)
@@ -76,5 +76,5 @@
   </link>
   <!-- ############################################################## macro robot's hip ####################################################-->
-  <xacro:macro name="hip" params='prefix reflect'>
+  <xacro:macro name="hip" params='prefix reflect member parent'>
     <link name="${prefix}_hip_link">
       <visual>
@@ -95,5 +95,5 @@
       <parent link="base_link"/>
       <child link="${prefix}_hip_link"/>
-      <origin xyz="${0.0305*reflect} 0 ${-(base_height+right_hip_height)/2}"/>
+      <origin xyz="${0.054*reflect} 0 ${-(base_height+right_hip_height)/2}"/>
     </joint>
   </xacro:macro>
@@ -101,6 +101,6 @@
   <xacro:hip prefix="left" reflect="-1"/>
   <!-- ############################################################## macro robot's bum ####################################################-->
-  <xacro:macro name="bum" params="prefix ">
-    <link name="${prefix}_bum_link">
+  <xacro:macro name="bum" params="prefix member parent z_origin">
+    <link name="${prefix}_${member}_link">
       <visual>
         <origin xyz="0 -0.0221 0"/>
@@ -116,13 +116,19 @@
       </collision>
     </link>
-    <joint name="${prefix}_hip_to_${prefix}_bum" type="fixed">
-      <parent link="${prefix}_hip_link"/>
-      <child link="${prefix}_bum_link"/>
-      <origin xyz="0 0 ${-right_bum_height/2}"/>
+    <joint name="${prefix}_${parent}_to_${prefix}_${member}" type="fixed">
+      <parent link="${prefix}_${parent}_link"/>
+      <child link="${prefix}_${member}_link"/>
+      <origin xyz="0 0 ${z_origin}"/>
     </joint>
       <!-- origin may been wong because 'z' may be not bum height divine by 2, it might increse in 'z' axis -->
   </xacro:macro>
-  <xacro:bum prefix="right"/>
-  <xacro:bum prefix="left"/>
+  <!-- right hip link to right bum link-->
+  <xacro:bum prefix="right" member="bum" parent="hip" z_origin="${-right_bum_height/2}"/>
+  <!-- left hip link to left bum link -->
+  <xacro:bum prefix="left" member="bum" parent="hip" z_origin="${-right_bum_height/2}"/>
+  <!-- right ankel link to right lower leg-->
+  <xacro:bum prefix="right" member="ankel" parent="lower_leg" z_origin="${-lower_leg_height}"/>
+  <!-- left ankel link to left lower leg -->
+  <xacro:bum prefix="left" member="ankel" parent="lower_leg" z_origin="${-lower_leg_height}"/>
   <!--########################################################## macro robot's upper leg #######################################################-->
   <xacro:macro name="upper_leg" params="prefix">
@@ -175,5 +181,5 @@
   <xacro:lower_leg prefix="left"/>
   <!--########################################################## macro robot's ankel #######################################################-->
-  <xacro:macro name="ankel" params="prefix">
+  <!-- <xacro:macro name="ankel" params="prefix">
     <link name="${prefix}_ankel_link">
       <visual>
@@ -197,5 +203,5 @@
   </xacro:macro>
   <xacro:ankel prefix="right"/>
-  <xacro:ankel prefix="left"/>
+  <xacro:ankel prefix="left"/> -->
 </robot>
   <!--########################################################## macro robot's upper foot #######################################################-->

Commit message: update fibot xacro
finish both leg

File: fibot_description/urdf/fibot_xacro.urdf.xacro (robot description, xacro)
@@ -28,4 +28,7 @@
   <xacro:property name="ankel_length" value="0.0922"/>
   <xacro:property name="ankel_height" value="0.06"/>
+  <xacro:property name="foot_width" value="0.09"/>
+  <xacro:property name="foot_length" value="0.165"/>
+  <xacro:property name="foot_height" value="0.027"/>
   <xacro:property name="pi" value="3.1415"/>
 <!-- ###########################################################set up property #################################################################-->
@@ -60,7 +63,16 @@
   </xacro:macro>
 <!-- add foot_print -->
+  <!-- <link name="foot_print">
+    <visual>
+      <origin xyz="0 0 0"/>
+      <geometry>
+        <box size="0 0 0"/>
+      </geometry>
+    </visual>
+  </link> -->
 <!-- add foot_print -->
   <link name="base_link">
     <visual>
+      <origin xyz="0 0 0"/>
       <geometry>
         <box size="${base_width} ${base_length} ${base_height}"/>
@@ -76,6 +88,6 @@
   </link>
   <!-- ############################################################## macro robot's hip ####################################################-->
-  <xacro:macro name="hip" params='prefix reflect member parent'>
-    <link name="${prefix}_hip_link">
+  <xacro:macro name="hip" params='prefix reflect member parent z_origin'>
+    <link name="${prefix}_${member}_link">
       <visual>
         <origin xyz="0 0 0"/>
@@ -92,12 +104,14 @@
       </collision>
     </link>
-    <joint name="base_link_to_${prefix}_hip_link" type="continuous">
-      <parent link="base_link"/>
-      <child link="${prefix}_hip_link"/>
-      <origin xyz="${0.054*reflect} 0 ${-(base_height+right_hip_height)/2}"/>
-    </joint>
-  </xacro:macro>
-  <xacro:hip prefix="right" reflect="1"/>
-  <xacro:hip prefix="left" reflect="-1"/>
+    <joint name="${parent}_to_${prefix}_${member}_link" type="continuous">
+      <parent link="${parent}"/>
+      <child link="${prefix}_${member}_link"/>
+      <origin xyz="${0.054*reflect} 0 ${z_origin}"/>
+    </joint>
+  </xacro:macro>
+  <xacro:hip prefix="right" reflect="1" member="hip" parent="base_link" z_origin="${-(base_height+right_hip_height)/2}"/>
+  <xacro:hip prefix="left" reflect="-1" member="hip" parent="base_link" z_origin="${-(base_height+right_hip_height)/2}"/>
+  <xacro:hip prefix="right" reflect="0" member="upper_foot" parent="right_ankel_link" z_origin="${-ankel_height/2}"/>
+  <xacro:hip prefix="left" reflect="0" member="upper_foot" parent="left_ankel_link" z_origin="${-ankel_height/2}"/>
   <!-- ############################################################## macro robot's bum ####################################################-->
   <xacro:macro name="bum" params="prefix member parent z_origin">
@@ -180,11 +194,11 @@
   <xacro:lower_leg prefix="right"/>
   <xacro:lower_leg prefix="left"/>
-  <!--########################################################## macro robot's ankel #######################################################-->
-  <!-- <xacro:macro name="ankel" params="prefix">
-    <link name="${prefix}_ankel_link">
-      <visual>
-        <origin xyz="0 -0.0221 0"/>
-        <geometry>
-          <box size="${ankel_width} ${ankel_length} ${ankel_height}"/>
+  <!--########################################################## macro robot's foot #######################################################-->
+  <xacro:macro name="foot" params="prefix reflect">
+    <link name="${prefix}_foot_link">
+      <visual>
+        <origin xyz="0 0 0"/>
+        <geometry>
+          <box size="${foot_width} ${foot_length} ${foot_height}"/>
         </geometry>
         <material name="turqouise"/>
@@ -192,16 +206,16 @@
       <collision>
         <geometry>
-          <box size="${ankel_width} ${ankel_length} ${ankel_height}"/>
-        </geometry>
-      </collision>
-    </link>
-    <joint name="${prefix}_lower_leg_to_${prefix}_ankel" type="fixed">
-      <parent link="${prefix}_lower_leg_link"/>
-      <child link="${prefix}_ankel_link"/>
-      <origin xyz="0 0 ${-lower_leg_height}"/>
-    </joint>
-  </xacro:macro>
-  <xacro:ankel prefix="right"/>
-  <xacro:ankel prefix="left"/> -->
+          <box size="${foot_width} ${foot_length} ${foot_height}"/>
+        </geometry>
+      </collision>
+    </link>
+    <joint name="${prefix}_upper_foot_to_${prefix}_foot" type="fixed">
+      <parent link="${prefix}_upper_foot_link"/>
+      <child link="${prefix}_foot_link"/>
+      <origin xyz="${0.018*reflect} -0.00989 0"/>
+    </joint>
+  </xacro:macro>
+  <xacro:foot prefix="right" reflect="1"/>
+  <xacro:foot prefix="left" reflect="-1"/>
 </robot>
   <!--########################################################## macro robot's upper foot #######################################################-->

Commit message: update launch file

File: fibot_description/urdf/fibot_xacro.urdf.xacro (robot description, xacro)
@@ -91,5 +91,5 @@
     <link name="${prefix}_${member}_link">
       <visual>
-        <origin xyz="0 0 0"/>
+        <origin xyz="0 0 0" rpy="0 0 0"/>
         <geometry>
           <box size="${right_hip_width} ${right_hip_length} ${right_hip_height}"/>
@@ -98,5 +98,5 @@
       </visual>
       <collision>
-        <origin xyz="0 0 0"/>
+        <origin xyz="0 0 0" rpy="0 0 0"/>
         <geometry>
           <box size="${right_hip_width} ${right_hip_length} ${right_hip_height}"/>
@@ -105,7 +105,8 @@
     </link>
     <joint name="${parent}_to_${prefix}_${member}_link" type="continuous">
+      <axis xyz="0 1 0" rpy="0 0 0"/>
       <parent link="${parent}"/>
       <child link="${prefix}_${member}_link"/>
-      <origin xyz="${0.054*reflect} 0 ${z_origin}"/>
+      <origin xyz="${0.054*reflect} 0 ${z_origin}" rpy="0 0 0"/>
     </joint>
   </xacro:macro>
